File: bargraph_demo.kicad_sch (KiCad schematic)
At the start: 0 parts

Commit message: update date and version number
Other:
- company: (none) -> @stoppattern
- title: (none) -> bargraph_demo
Changed lines of the file:
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@@
 	(generator_version "10.0")
 	(paper "A4")
+	(title_block
+		(title "bargraph_demo")
+		(date "%%date%%")
+		(rev "%%version%%")
+		(company "@stoppattern")
+		(comment 1 "651系 速度計 デモ基板")
+	)
 	(sheet_instances
 		(path "/"

Commit message: update sch
Parts:
- added C1: 1u, Capacitor_SMD:C_0603_1608Metric, symbol Device:C
- added C2, C3, C5, C6, C8, C9: 0.1u, Capacitor_SMD:C_0402_1005Metric, symbol Device:C
- added C4: 4.7u, Capacitor_SMD:C_0603_1608Metric, symbol Device:C
- added C7: 22u, Capacitor_SMD:C_0603_1608Metric, symbol Device:C
- added D1: 3.3V, LED_SMD:LED_0603_1608Metric, symbol Device:LED
- added D2: RX, LED_SMD:LED_0603_1608Metric, symbol Device:LED
- added D3: TX, LED_SMD:LED_0603_1608Metric, symbol Device:LED
- added D4: IO16, LED_SMD:LED_0603_1608Metric, symbol Device:LED
- added D5: IO17, LED_SMD:LED_0603_1608Metric, symbol Device:LED
- added D6, D7: IO18, LED_SMD:LED_0603_1608Metric, symbol Device:LED
- added D8, D9: IO19, LED_SMD:LED_0603_1608Metric, symbol Device:LED
- added J1: USB_C_Receptacle_USB2.0_16P, Connector_USB:USB_C_Receptacle_GCT_USB4105-xx-A_16P_TopMnt_Horizontal, symbol Connector:USB_C_Receptacle_USB2.0_16P
- added J2: Barrel_Jack_Switch, Connector_BarrelJack:BarrelJack_Kycon_KLDX-0202-xC_Horizontal, symbol Connector:Barrel_Jack_Switch
- added J3: VR, Connector_JST:JST_XA_B03B-XASK-1_1x03_P2.50mm_Vertical, symbol Connector_Generic:Conn_01x03
- added J4: LCD, symbol Connector_Generic:Conn_01x08
- added JP1: CFG1, Jumper:SolderJumper-3_P1.3mm_Open_RoundedPad1.0x1.5mm, symbol Jumper:SolderJumper_3_Open
- added JP2: CFG2, Jumper:SolderJumper-3_P1.3mm_Open_RoundedPad1.0x1.5mm, symbol Jumper:SolderJumper_3_Open
- added JP3: CFG3, Jumper:SolderJumper-3_P1.3mm_Open_RoundedPad1.0x1.5mm, symbol Jumper:SolderJumper_3_Open
- added Q1, Q2, Q3, Q4: BSS138, Package_TO_SOT_SMD:SOT-23, symbol Transistor_FET:BSS138
- added R1: 10k, Resistor_SMD:R_0603_1608Metric, symbol Device:R
- added R10, R11, R12, R13, R14, R15, R2, R3, R4, R5, R8, R9: 1k, Resistor_SMD:R_0603_1608Metric, symbol Device:R
- added R6, R7: 0, Resistor_SMD:R_0603_1608Metric, symbol Device:R
- added RV1: VR, symbol Device:R_Potentiometer
- added SW1: IO0, Button_Switch_SMD:SW_Push_SPST_NO_Alps_SKRK, symbol Switch:SW_Push
- added SW2: RST, Button_Switch_SMD:SW_Push_SPST_NO_Alps_SKRK, symbol Switch:SW_Push
- added SW3: RotaryEncoder_Switch, symbol Device:RotaryEncoder_Switch
- added U1: CH224K, Package_SO:SSOP-10-1EP_3.9x4.9mm_P1mm_EP2.1x3.3mm, symbol Interface_USB:CH224K
- added U2: R-78E3.3-1.0, Converter_DCDC:Converter_DCDC_RECOM_R-78E-0.5_THT, symbol Converter_DCDC:R-78E3.3-1.0
- added U3: CP2102N-Axx-xQFN28, Package_DFN_QFN:QFN-28-1EP_5x5mm_P0.5mm_EP3.35x3.35mm, symbol Interface_USB:CP2102N-Axx-xQFN28
- added U4: ESP32-WROOM-32E, RF_Module:ESP32-WROOM-32E, symbol RF_Module:ESP32-WROOM-32E
Connections:
- new net: D6.1 (K), D7.1 (K), Q3.3 (D)
- new net: D7.2 (A), R13.1
- new net: Q2.1 (G), R7.1
- new net: D4.2 (A), R10.1
- new net: D6.2 (A), R12.1
- new net: JP2.2 (C), U1.2 (CFG2)
- new net: D8.1 (K), D9.1 (K), Q4.3 (D)
- new net: D9.2 (A), R15.1
- new net: Q1.1 (G), R6.1
- new net: JP3.2 (C), U1.3 (CFG3)
- new net: D5.2 (A), R11.1
- new net: JP1.2 (C), U1.9 (CFG1)
- new net: D8.2 (A), R14.1
- new net: D1.2 (A), R5.1
- new net: D3.2 (A), R9.1
- new net: D2.2 (A), R8.1
- new net: R1.2, U1.8 (VBUS)
- new net +3V3: C1.1, C4.1, C5.1, C7.1, C8.1, J3.3 (Pin_3), JP1.1 (A), JP2.1 (A), JP3.1 (A), R12.2, R13.2, R14.2, R15.2, R2.2, R3.2, R4.2, R5.2, R8.2, R9.2, RV1.1, U1.1 (VDD), U2.3 (OUT), U3.6 (VDD), U3.7 (VREGIN), U3.9 (~{RST}), U4.2 (VDD)
- new net CC1: J1.A5 (CC1), U1.7 (CC1)
- new net CC2: J1.B5 (CC2), U1.6 (CC2)
- new net D+: J1.A6 (D+), J1.B6 (D+), U3.4 (D+)
- new net D-: J1.A7 (D-), J1.B7 (D-), U3.5 (D-)
- new net EN: C3.1, C6.1, Q1.3 (D), R4.1, SW2.2, U4.3 (EN)
- new net GND: C1.2, C2.2, C3.2, C4.2, C5.2, C6.2, C7.2, C8.2, D1.1 (K), D4.1 (K), D5.1 (K), J1.A1 (GND), J1.A12 (GND), J1.B1 (GND), J1.B12 (GND), J3.1 (Pin_1), JP1.3 (B), JP2.3 (B), JP3.3 (B), Q3.2 (S), Q4.2 (S), RV1.3, SW1.1, SW2.1, U1.11 (GND), U2.2 (GND), U3.29 (GND), U3.3 (GND), U4.1 (GND), U4.15 (GND), U4.38 (GND), U4.39 (GND)
- new net GNDD: J2.2, J2.3
- new net IO0: C2.1, Q2.3 (D), R3.1, SW1.2, U4.25 (IO0)
- new net IO13: J3.2 (Pin_2), RV1.2, U4.16 (IO13)
- new net IO16: R10.2, U4.27 (IO16)
- new net IO17: R11.2, U4.28 (IO17)
- new net IO18: Q3.1 (G), U4.30 (IO18)
- new net IO19: Q4.1 (G), U4.31 (IO19)
- new net RX: U3.26 (TXD), U4.34 (RXD0/IO3)
- new net TX: U3.25 (RXD), U4.35 (TXD0/IO1)
- new net VBUS: J1.A4 (VBUS), J1.A9 (VBUS), J1.B4 (VBUS), J1.B9 (VBUS), R1.1, R2.1, U2.1 (IN)
- new net VCC: J2.1
- new net ~{DTR}: Q2.2 (S), R6.2, U3.28 (~{DTR})
- new net ~{RTS}: Q1.2 (S), R7.2, U3.24 (~{RTS})
- new net ~{RXT}: D2.1 (K), U3.19 (~{TXT}/GPIO.0)
- new net ~{TXT}: D3.1 (K), U3.18 (~{RXT}/GPIO.1)
- no-connect marks 0 -> 29
Other:
- note added: "Automatic Download"
- note added: "CC Controller"
- note added: "DC/DC Converter"
- note added: "ESP32"
- note added: "Green POW"
- note added: "Input - Analog"
- note added: "Input - Switch"
- note added: "Output - LED"
- note added: "Output - Serial"
- note added: "Power"
- note added: "Power Flag"
- note added: "Pull-up"
- note added: "Red"
- note added: "USB-C"
- note added: "USB/Serial Converter"
- note added: "VBUS: 15V"
- note added: "White"
- note added: "Yellow"
